Commit message: Save local gimbalrotor changes

File: robots/gimbalrotor/robots/beetle_hyper/gimbalrotor.urdf.xacro (robot description, xacro)
@@ -5,6 +5,6 @@
   <xacro:include filename="$(find gimbalrotor)/urdf/beetle_hyper/common.xacro" />
   <xacro:gimbalrotor_center_link child1="1" child2="2" child3="3" child4="4"/>
-  <xacro:gimbalrotor_thrust_link self="1" rotor_direction="-1"/>
-  <xacro:gimbalrotor_thrust_link self="2" rotor_direction="1"/>
+  <xacro:gimbalrotor_thrust_link self="1" rotor_direction="1"/>
+  <xacro:gimbalrotor_thrust_link self="2" rotor_direction="-1"/>
   <xacro:gimbalrotor_thrust_link self="3" rotor_direction="-1"/>
   <xacro:gimbalrotor_thrust_link self="4" rotor_direction="1"/>

File: robots/gimbalrotor/urdf/beetle_hyper/gimbalrotor.urdf.xacro (robot description, xacro)
@@ -24,5 +24,6 @@
       <inertial>
         <origin xyz="0.0257171 0.0007358  0.0813823" rpy="0 0 0"/>
-        <mass value="2.8200834"/>
+        <!-- <mass value="2.8200834"/> -->
+	<mass value="2.0200834"/>
         <inertia
             ixx="0.0679394" iyy="0.1142367" izz="0.1213159"
@@ -82,8 +83,8 @@
     </xacro:macro>
     ## dummy rotor arms
-    <xacro:dummy_rotor_arm id = "${child1}" x = "0.12041" y="0.12041" z = "0.0555" yaw = "${pi/4.0}"/>
+    <xacro:dummy_rotor_arm id = "${child1}" x = "-0.12041" y="-0.12041" z = "0.0555" yaw = "${-pi*3/4.0}"/>
     <xacro:dummy_rotor_arm id = "${child2}" x = "-0.12129" y="0.12150" z = "0.0555" yaw = "${pi*3.0/4.0}"/>
-    <xacro:dummy_rotor_arm id = "${child3}" x = "-0.12129" y="-0.12150" z = "0.0555" yaw = "${pi*5.0/4.0}"/>
-    <xacro:dummy_rotor_arm id = "${child4}" x = "0.12129" y="-0.12150" z = "0.0555" yaw = "${-pi/4.0}"/>
+    <xacro:dummy_rotor_arm id = "${child3}" x = "0.12129" y="-0.12150" z = "0.0555" yaw = "${-pi/4.0}"/>
+    <xacro:dummy_rotor_arm id = "${child4}" x = "0.12129" y="0.12150" z = "0.0555" yaw = "${pi/4.0}"/>
     ## dummy link for the contact point coordinate
       <link name="contact_point">
@@ -111,5 +112,5 @@
       <inertial>
         <origin xyz="0.0223521 0.0 0.00776312" rpy="0 0 0"/>
-        <mass value="0.15944"/>
+p        <mass value="0.15944"/>
         <inertia
             ixx="0.00007458" iyy="0.00007325" izz="0.00007756"
