Commit message: gazebo linkname&mass

File: robots/gimbalrotor/urdf/beetle_hyper/common.xacro (robot description, xacro)
@@ -10,5 +10,5 @@
   <!-- friction -->
   <xacro:macro name="friction" params="self">
-    <gazebo reference="link${self}">
+    <gazebo reference="${self}">
       <mu1>0.1</mu1>
       <mu2>0.1</mu2>

File: robots/gimbalrotor/urdf/beetle_hyper/gimbalrotor.urdf.xacro (robot description, xacro)
@@ -110,5 +110,5 @@
 	  <!-- hook_tool_link原点から見た重心位置 -->
 	  <origin xyz="0 0 0" rpy="0 0 0"/>
-	  <mass value="0.01"/>
+	  <mass value="0.0001"/>
 	  <inertia
 	      ixx="8.309234e-4" ixy="-3.962e-8" ixz="5.48e-9"
