Commit message: for terrestrial_docking

File: robots/gimbalrotor/urdf/beetle_hyper/gimbalrotor.urdf.xacro (robot description, xacro)
@@ -102,6 +102,46 @@
         <origin rpy="0 0 0" xyz="0.26 0 0"/>
         <axis xyz="0 0 1"/>
-      </joint>
-    <xacro:friction self="base_link"/>
+	<limit lower="0" upper="0" effort="0" velocity="0"/>
+      </joint>
+      <xacro:friction self="base_link"/>
+      <!-- hook tool -->
+      <link name="hook_tool_link">
+	<inertial>
+	  <!-- hook_tool_link原点から見た重心位置 -->
+	  <origin xyz="0 0 0" rpy="0 0 0"/>
+	  <mass value="0.01"/>
+	  <inertia
+	      ixx="8.309234e-4" ixy="-3.962e-8" ixz="5.48e-9"
+	      iyy="3.7551831e-4" iyz="-1.77238e-4"
+	      izz="5.5049843e-4"/>
+	</inertial>
+	<!-- <visual> -->
+	<!--   <origin xyz="0 0 0" rpy="0 0 0"/> -->
+	<!--   <geometry> -->
+	<!--     <mesh filename="package://gimbalrotor/src/model/untitled.stl" -->
+	<!-- 	  scale="0.001 0.001 0.001"/> -->
+	<!--   </geometry> -->
+	<!-- </visual> -->
+	<collision>
+	  <origin xyz="0 0 0" rpy="0 0 0"/>
+	  <geometry>
+	    <mesh filename="package://gimbalrotor/src/model/untitled.stl"
+		  scale="0.001 0.001 0.001"/>
+	  </geometry>
+	</collision>
+      </link>
+      <joint name="hook_tool_joint" type="fixed">
+	<parent link="base_link"/>
+	<child link="hook_tool_link"/>
+	<origin xyz="0.2575 0 0.09141" rpy="0 0 0"/>
+      </joint>
+      <gazebo reference="hook_tool_joint">
+	<preserveFixedJoint>true</preserveFixedJoint>
+      </gazebo>
+      <gazebo reference="hook_tool_link">
+	<!-- <preserveFixedJoint>true</preserveFixedJoint> -->
+	<mu1>0.1</mu1>
+	<mu2>0.1</mu2>
+      </gazebo>
   </xacro:macro>
   <xacro:macro name="gimbalrotor_thrust_link" params="self rotor_direction">

Commit message: urdfundo PIDgain

File: robots/gimbalrotor/urdf/beetle_hyper/gimbalrotor.urdf.xacro (robot description, xacro)
@@ -24,5 +24,6 @@
       <inertial>
         <origin xyz="0.0257171 0.0007358  0.0813823" rpy="0 0 0"/>
-        <mass value="2.8200834"/>
+        <!-- <mass value="2.8200834"/> -->
+	<mass value="2.0200834"/>
         <inertia
             ixx="0.0679394" iyy="0.1142367" izz="0.1213159"
@@ -105,43 +106,43 @@
       </joint>
       <xacro:friction self="base_link"/>
-      <!-- hook tool -->
-      <link name="hook_tool_link">
-	<inertial>
-	  <!-- hook_tool_link原点から見た重心位置 -->
-	  <origin xyz="0 0 0" rpy="0 0 0"/>
-	  <mass value="0.0001"/>
-	  <inertia
-	      ixx="8.309234e-4" ixy="-3.962e-8" ixz="5.48e-9"
-	      iyy="3.7551831e-4" iyz="-1.77238e-4"
-	      izz="5.5049843e-4"/>
-	</inertial>
-	<!-- <visual> -->
-	<!--   <origin xyz="0 0 0" rpy="0 0 0"/> -->
-	<!--   <geometry> -->
-	<!--     <mesh filename="package://gimbalrotor/src/model/untitled.stl" -->
-	<!-- 	  scale="0.001 0.001 0.001"/> -->
-	<!--   </geometry> -->
-	<!-- </visual> -->
-	<collision>
-	  <origin xyz="0 0 0" rpy="0 0 0"/>
-	  <geometry>
-	    <mesh filename="package://gimbalrotor/src/model/untitled.stl"
-		  scale="0.001 0.001 0.001"/>
-	  </geometry>
-	</collision>
-      </link>
-      <joint name="hook_tool_joint" type="fixed">
-	<parent link="base_link"/>
-	<child link="hook_tool_link"/>
-	<origin xyz="0.2575 0 0.09141" rpy="0 0 0"/>
-      </joint>
-      <gazebo reference="hook_tool_joint">
-	<preserveFixedJoint>true</preserveFixedJoint>
-      </gazebo>
-      <gazebo reference="hook_tool_link">
-	<!-- <preserveFixedJoint>true</preserveFixedJoint> -->
-	<mu1>0.1</mu1>
-	<mu2>0.1</mu2>
-      </gazebo>
+      <!-- <!-\- hook tool -\-> -->
+      <!-- <link name="hook_tool_link"> -->
+      <!-- 	<inertial> -->
+      <!-- 	  <!-\- hook_tool_link原点から見た重心位置 -\-> -->
+      <!-- 	  <origin xyz="0 0 0" rpy="0 0 0"/> -->
+      <!-- 	  <mass value="0.0001"/> -->
+      <!-- 	  <inertia -->
+      <!-- 	      ixx="8.309234e-4" ixy="-3.962e-8" ixz="5.48e-9" -->
+      <!-- 	      iyy="3.7551831e-4" iyz="-1.77238e-4" -->
+      <!-- 	      izz="5.5049843e-4"/> -->
+      <!-- 	</inertial> -->
+      <!-- 	<!-\- <visual> -\-> -->
+      <!-- 	<!-\-   <origin xyz="0 0 0" rpy="0 0 0"/> -\-> -->
+      <!-- 	<!-\-   <geometry> -\-> -->
+      <!-- 	<!-\-     <mesh filename="package://gimbalrotor/src/model/untitled.stl" -\-> -->
+      <!-- 	<!-\- 	  scale="0.001 0.001 0.001"/> -\-> -->
+      <!-- 	<!-\-   </geometry> -\-> -->
+      <!-- 	<!-\- </visual> -\-> -->
+      <!-- 	<collision> -->
+      <!-- 	  <origin xyz="0 0 0" rpy="0 0 0"/> -->
+      <!-- 	  <geometry> -->
+      <!-- 	    <mesh filename="package://gimbalrotor/src/model/untitled.stl" -->
+      <!-- 		  scale="0.001 0.001 0.001"/> -->
+      <!-- 	  </geometry> -->
+      <!-- 	</collision> -->
+      <!-- </link> -->
+      <!-- <joint name="hook_tool_joint" type="fixed"> -->
+      <!-- 	<parent link="base_link"/> -->
+      <!-- 	<child link="hook_tool_link"/> -->
+      <!-- 	<origin xyz="0.2575 0 0.09141" rpy="0 0 0"/> -->
+      <!-- </joint> -->
+      <!-- <gazebo reference="hook_tool_joint"> -->
+      <!-- 	<preserveFixedJoint>true</preserveFixedJoint> -->
+      <!-- </gazebo> -->
+      <!-- <gazebo reference="hook_tool_link"> -->
+      <!-- 	<!-\- <preserveFixedJoint>true</preserveFixedJoint> -\-> -->
+      <!-- 	<mu1>0.1</mu1> -->
+      <!-- 	<mu2>0.1</mu2> -->
+      <!-- </gazebo> -->
   </xacro:macro>
   <xacro:macro name="gimbalrotor_thrust_link" params="self rotor_direction">
