Commit message: changed python

File: robots/gimbalrotor/urdf/beetle_hyper/gimbalrotor.urdf.xacro (robot description, xacro)
@@ -25,5 +25,5 @@
         <origin xyz="0.0257171 0.0007358  0.0813823" rpy="0 0 0"/>
         <!-- <mass value="2.8200834"/> -->
-	<mass value="2.0200834"/>
+	<mass value="3.0200834"/>
         <inertia
             ixx="0.0679394" iyy="0.1142367" izz="0.1213159"
@@ -106,43 +106,43 @@
       </joint>
       <xacro:friction self="base_link"/>
-      <!-- <!-\- hook tool -\-> -->
-      <!-- <link name="hook_tool_link"> -->
-      <!-- 	<inertial> -->
-      <!-- 	  <!-\- hook_tool_link原点から見た重心位置 -\-> -->
-      <!-- 	  <origin xyz="0 0 0" rpy="0 0 0"/> -->
-      <!-- 	  <mass value="0.0001"/> -->
-      <!-- 	  <inertia -->
-      <!-- 	      ixx="8.309234e-4" ixy="-3.962e-8" ixz="5.48e-9" -->
-      <!-- 	      iyy="3.7551831e-4" iyz="-1.77238e-4" -->
-      <!-- 	      izz="5.5049843e-4"/> -->
-      <!-- 	</inertial> -->
-      <!-- 	<!-\- <visual> -\-> -->
-      <!-- 	<!-\-   <origin xyz="0 0 0" rpy="0 0 0"/> -\-> -->
-      <!-- 	<!-\-   <geometry> -\-> -->
-      <!-- 	<!-\-     <mesh filename="package://gimbalrotor/src/model/untitled.stl" -\-> -->
-      <!-- 	<!-\- 	  scale="0.001 0.001 0.001"/> -\-> -->
-      <!-- 	<!-\-   </geometry> -\-> -->
-      <!-- 	<!-\- </visual> -\-> -->
-      <!-- 	<collision> -->
-      <!-- 	  <origin xyz="0 0 0" rpy="0 0 0"/> -->
-      <!-- 	  <geometry> -->
-      <!-- 	    <mesh filename="package://gimbalrotor/src/model/untitled.stl" -->
-      <!-- 		  scale="0.001 0.001 0.001"/> -->
-      <!-- 	  </geometry> -->
-      <!-- 	</collision> -->
-      <!-- </link> -->
-      <!-- <joint name="hook_tool_joint" type="fixed"> -->
-      <!-- 	<parent link="base_link"/> -->
-      <!-- 	<child link="hook_tool_link"/> -->
-      <!-- 	<origin xyz="0.2575 0 0.09141" rpy="0 0 0"/> -->
-      <!-- </joint> -->
-      <!-- <gazebo reference="hook_tool_joint"> -->
-      <!-- 	<preserveFixedJoint>true</preserveFixedJoint> -->
-      <!-- </gazebo> -->
-      <!-- <gazebo reference="hook_tool_link"> -->
-      <!-- 	<!-\- <preserveFixedJoint>true</preserveFixedJoint> -\-> -->
-      <!-- 	<mu1>0.1</mu1> -->
-      <!-- 	<mu2>0.1</mu2> -->
-      <!-- </gazebo> -->
+      <!-- hook tool -->
+      <link name="hook_tool_link">
+	<inertial>
+	  <!-- hook_tool_link原点から見た重心位置 -->
+	  <origin xyz="0 0 0" rpy="0 0 0"/>
+	  <mass value="0.0001"/>
+	  <inertia
+	      ixx="8.309234e-4" ixy="-3.962e-8" ixz="5.48e-9"
+	      iyy="3.7551831e-4" iyz="-1.77238e-4"
+	      izz="5.5049843e-4"/>
+	</inertial>
+	<!-- <visual> -->
+	<!--   <origin xyz="0 0 0" rpy="0 0 0"/> -->
+	<!--   <geometry> -->
+	<!--     <mesh filename="package://gimbalrotor/src/model/untitled.stl" -->
+	<!-- 	  scale="0.001 0.001 0.001"/> -->
+	<!--   </geometry> -->
+	<!-- </visual> -->
+	<collision>
+	  <origin xyz="0 0 0" rpy="0 0 0"/>
+	  <geometry>
+	    <mesh filename="package://gimbalrotor/src/model/untitled.stl"
+		  scale="0.001 0.001 0.001"/>
+	  </geometry>
+	</collision>
+      </link>
+      <joint name="hook_tool_joint" type="fixed">
+	<parent link="base_link"/>
+	<child link="hook_tool_link"/>
+	<origin xyz="0.2575 0 0.09141" rpy="0 0 0"/>
+      </joint>
+      <gazebo reference="hook_tool_joint">
+	<preserveFixedJoint>true</preserveFixedJoint>
+      </gazebo>
+      <gazebo reference="hook_tool_link">
+	<!-- <preserveFixedJoint>true</preserveFixedJoint> -->
+	<mu1>0.1</mu1>
+	<mu2>0.1</mu2>
+      </gazebo>
   </xacro:macro>
   <xacro:macro name="gimbalrotor_thrust_link" params="self rotor_direction">

Commit message: change yaml gimabalrotor.urdf

File: robots/gimbalrotor/urdf/beetle_hyper/gimbalrotor.urdf.xacro (robot description, xacro)
@@ -109,39 +109,40 @@
       <link name="hook_tool_link">
 	<inertial>
-	  <!-- hook_tool_link原点から見た重心位置 -->
-	  <origin xyz="0 0 0" rpy="0 0 0"/>
-	  <mass value="0.0001"/>
-	  <inertia
-	      ixx="8.309234e-4" ixy="-3.962e-8" ixz="5.48e-9"
-	      iyy="3.7551831e-4" iyz="-1.77238e-4"
-	      izz="5.5049843e-4"/>
-	</inertial>
-	<!-- <visual> -->
-	<!--   <origin xyz="0 0 0" rpy="0 0 0"/> -->
-	<!--   <geometry> -->
-	<!--     <mesh filename="package://gimbalrotor/src/model/untitled.stl" -->
-	<!-- 	  scale="0.001 0.001 0.001"/> -->
-	<!--   </geometry> -->
-	<!-- </visual> -->
-	<collision>
-	  <origin xyz="0 0 0" rpy="0 0 0"/>
-	  <geometry>
-	    <mesh filename="package://gimbalrotor/src/model/untitled.stl"
-		  scale="0.001 0.001 0.001"/>
-	  </geometry>
-	</collision>
+      	  <!-- hook_tool_link原点から見た重心位置 -->
+      	  <origin xyz="0 0 0" rpy="0 0 0"/>
+      	  <mass value="0.0001"/>
+      	  <inertia
+      	      ixx="8.309234e-4" ixy="-3.962e-8" ixz="5.48e-9"
+      	      iyy="3.7551831e-4" iyz="-1.77238e-4"
+      	      izz="5.5049843e-4"/>
+      	</inertial>
+      	<!-- <visual> -->
+      	<!--   <origin xyz="0 0 0" rpy="0 0 0"/> -->
+      	<!--   <geometry> -->
+      	<!--     <mesh filename="package://gimbalrotor/src/model/untitled.stl" -->
+      	<!-- 	  scale="0.001 0.001 0.001"/> -->
+      	<!--   </geometry> -->
+      	<!-- </visual> -->
+      	<collision>
+      	  <origin xyz="0 0 0" rpy="0 0 0"/>
+      	  <geometry>
+      	    <mesh filename="package://gimbalrotor/src/model/untitled.stl"
+      		  scale="0.001 0.001 0.001"/>
+      	  </geometry>
+      	</collision>
       </link>
       <joint name="hook_tool_joint" type="fixed">
-	<parent link="base_link"/>
-	<child link="hook_tool_link"/>
-	<origin xyz="0.2575 0 0.09141" rpy="0 0 0"/>
+      	<parent link="base_link"/>
+      	<child link="hook_tool_link"/>
+      	<origin xyz="0.2575 0 0.09141" rpy="0 0 0"/>
       </joint>
       <gazebo reference="hook_tool_joint">
-	<preserveFixedJoint>true</preserveFixedJoint>
+      	<preserveFixedJoint>true</preserveFixedJoint>
       </gazebo>
       <gazebo reference="hook_tool_link">
-	<!-- <preserveFixedJoint>true</preserveFixedJoint> -->
-	<mu1>0.1</mu1>
-	<mu2>0.1</mu2>
+      	<!-- <preserveFixedJoint>true</preserveFixedJoint> -->
+      	<mu1>0.1</mu1>
+      	<mu2>0.1</mu2>
+>>>>>>> Stashed changes
       </gazebo>
   </xacro:macro>

Commit message: add box and change machine model ver1

File: robots/gimbalrotor/urdf/beetle_hyper/gimbalrotor.urdf.xacro (robot description, xacro)
@@ -23,22 +23,55 @@
     <link name="base_link">
       <inertial>
-        <origin xyz="0.0257171 0.0007358  0.0813823" rpy="0 0 0"/>
+        <!-- <origin xyz="0.0257171 0.0007358  0.0813823" rpy="0 0 0"/> -->
         <!-- <mass value="2.8200834"/> -->
+	<origin xyz="0.0225071 0.0006440 0.0696371" rpy="0 0 0"/>
 	<mass value="3.0200834"/>
-        <inertia
-            ixx="0.0679394" iyy="0.1142367" izz="0.1213159"
-            ixy="-0.0001621" ixz="0.00612466" iyz="0.0000964"/>
+	<inertia
+	    ixx="0.0625427" ixy="-0.0002088" ixz="0.0010742"
+	    iyy="0.1072134" iyz="-0.0000481" izz="0.1375859"/>
+        <!-- <inertia -->
+        <!--     ixx="0.0679394" iyy="0.1142367" izz="0.1213159" -->
+        <!--     ixy="-0.0001621" ixz="0.00612466" iyz="0.0000964"/> -->
       </inertial>
       <visual>
         <origin xyz="0 0 0" rpy="0 0 3.141592"/>
         <geometry>
-          <mesh filename="package://gimbalrotor/urdf/beetle_hyper/mesh/base_link_hyper.dae"/>
+          <!-- <mesh filename="package://gimbalrotor/urdf/beetle_hyper/mesh/base_link_hyper.dae"/> -->
+	  <mesh filename="package://gimbalrotor/urdf/beetle_hyper/mesh/Beetle_hyper_terrestrial.STL"
+		scale="0.001 0.001 0.001"/>
         </geometry>
       </visual>
-      <collision>
-        <origin xyz="0 0 0.053" rpy="0 0 0"/>
-        <geometry>
-          <box size="0.52 0.52 0.241"/>
-        </geometry>
+      <!-- <collision> -->
+        <!-- <origin xyz="0 0 0.053" rpy="0 0 0"/> -->
+        <!-- <geometry> -->
+        <!--   <box size="0.52 0.52 0.241"/> -->
+        <!-- </geometry> -->
+      <!-- </collision> -->
+      <collision name="base_collision_front">
+	<origin xyz="0.13 0 0.053" rpy="0 0 0"/>
+	<geometry>
+	  <box size="0.26 0.52 0.241"/>
+	</geometry>
+      </collision>
+      <!-- 後方左側 -->
+      <collision name="base_collision_rear_left">
+	<origin xyz="-0.13 0.155 0.053" rpy="0 0 0"/>
+	<geometry>
+	  <box size="0.26 0.21 0.241"/>
+	</geometry>
+      </collision>
+      <!-- 後方右側 -->
+      <collision name="base_collision_rear_right">
+	<origin xyz="-0.13 -0.155 0.053" rpy="0 0 0"/>
+	<geometry>
+	  <box size="0.26 0.21 0.241"/>
+	</geometry>
+      </collision>
+      <collision name="female_head_collision">
+      	<origin xyz="-0.23506 0 0.148" rpy="0 0 0"/>
+      	  <geometry>
+      	    <mesh filename="package://gimbalrotor/src/model/female_head_collision.STL"
+      		  scale="0.001 0.001 0.001"/>
+      	  </geometry>
       </collision>
     </link>
@@ -112,8 +145,12 @@
       	  <origin xyz="0 0 0" rpy="0 0 0"/>
       	  <mass value="0.0001"/>
-      	  <inertia
-      	      ixx="8.309234e-4" ixy="-3.962e-8" ixz="5.48e-9"
-      	      iyy="3.7551831e-4" iyz="-1.77238e-4"
-      	      izz="5.5049843e-4"/>
+      	  <!-- <inertia -->
+      	  <!--     ixx="8.309234e-4" ixy="-3.962e-8" ixz="5.48e-9" -->
+      	  <!--     iyy="3.7551831e-4" iyz="-1.77238e-4" -->
+      	  <!--     izz="5.5049843e-4"/> -->
+	  <inertia
+              ixx="0.000001" ixy="0.0" ixz="0.0"
+              iyy="0.0001" iyz="0.0"
+              izz="0.0001"/>
       	</inertial>
       	<!-- <visual> -->
@@ -144,7 +181,107 @@
       	<mu1>0.1</mu1>
       	<mu2>0.1</mu2>
->>>>>>> Stashed changes
       </gazebo>
-  </xacro:macro>
+      <xacro:property name="caster_radius" value="0.0047625"/>
+      <xacro:property name="caster_center_z" value="-0.0787375"/>
+      <xacro:macro name="ball_caster_contact" params="id x y">
+	<link name="ball_caster_${id}">
+	  <inertial>
+	    <origin xyz="0 0 0" rpy="0 0 0"/>
+	    <mass value="0.0001"/>
+	    <inertia
+		ixx="1e-5"
+		iyy="1e-5"
+		izz="1e-5"
+		ixy="0"
+		ixz="0"
+		iyz="0"/>
+	  </inertial>
+	  <collision>
+	    <origin xyz="0 0 0" rpy="0 0 0"/>
+	    <geometry>
+              <sphere radius="${caster_radius}"/>
+	    </geometry>
+	  </collision>
+	</link>
+	<!-- <link name="ball_caster_x_${id}"> -->
+	<!--   <inertial> -->
+	<!--     <origin xyz="0 0 0" rpy="0 0 0"/> -->
+	<!--     <mass value="0.00001"/> -->
+	<!--     <inertia -->
+	<!-- 	ixx="1e-5" -->
+	<!-- 	iyy="1e-5" -->
+	<!-- 	izz="1e-5" -->
+	<!-- 	ixy="0" -->
+	<!-- 	ixz="0" -->
+	<!-- 	iyz="0"/> -->
+	<!--   </inertial> -->
+	<!-- </link> -->
+	<!-- <joint name="ball_caster_x_joint_${id}" type="continuous"> -->
+	<!--   <parent link="base_link"/> -->
+	<!--   <child link="ball_caster_x_${id}"/> -->
+	<!--   <origin -->
+	<!--       xyz="${x} ${y} ${caster_center_z}" -->
+	<!--       rpy="0 0 0"/> -->
+	<!--   <axis xyz="1 0 0"/> -->
+	<!--   <dynamics -->
+	<!--       damping="0.0001" -->
+	<!--       friction="0.0"/> -->
+	<!-- </joint> -->
+	<!-- <link name="ball_caster_y_${id}"> -->
+	<!--   <inertial> -->
+	<!--     <origin xyz="0 0 0" rpy="0 0 0"/> -->
+	<!--     <mass value="0.00001"/> -->
+	<!--     <inertia -->
+	<!-- 	ixx="1e-5" -->
+	<!-- 	iyy="1e-5" -->
+	<!-- 	izz="1e-5" -->
+	<!-- 	ixy="0" -->
+	<!-- 	ixz="0" -->
+	<!-- 	iyz="0"/> -->
+	<!--   </inertial> -->
+	<!-- </link> -->
+	<!-- <joint name="ball_caster_y_joint_${id}" type="continuous"> -->
+	<!--   <parent link="ball_caster_x_${id}"/> -->
+	<!--   <child link="ball_caster_y_${id}"/> -->
+	<!--   <origin xyz="0 0 0" rpy="0 0 0"/> -->
+	<!--   <axis xyz="0 1 0"/> -->
+	<!--   <dynamics -->
+	<!--       damping="0.0001" -->
+	<!--       friction="0.0"/> -->
+	<!-- </joint> -->
+	<!-- <joint name="ball_caster_z_joint_${id}" type="continuous"> -->
+	<!--   <parent link="ball_caster_y_${id}"/> -->
+	<!--   <child link="ball_caster_${id}"/> -->
+	<!--   <origin xyz="0 0 0" rpy="0 0 0"/> -->
+	<!--   <axis xyz="0 0 1"/> -->
+	<!--   <dynamics -->
+	<!--       damping="0.0001" -->
+	<!--       friction="0.0"/> -->
+	<!-- </joint> -->
+	<joint name="ball_caster_${id}_joint" type="fixed">
+	  <parent link="base_link"/>
+	  <child link="ball_caster_${id}"/>
+	  <origin
+	      xyz="${x} ${y} ${caster_center_z}"
+	      rpy="0 0 0"/>
+	</joint>
+	<gazebo reference="ball_caster_${id}">
+	  <mu1>0.01</mu1>
+	  <mu2>0.01</mu2>
+	  <kp>1000000.0</kp>
+	  <kd>100.0</kd>
+	  <minDepth>0.0005</minDepth>
+	  <maxVel>0.1</maxVel>
+	</gazebo>
+      </xacro:macro>
+      <xacro:ball_caster_contact id="1" x="0.240594"  y="0.240594"/>
+      <xacro:ball_caster_contact id="2" x="-0.240594" y="0.240594"/>
+      <xacro:ball_caster_contact id="3" x="-0.240594" y="-0.240594"/>
+      <xacro:ball_caster_contact id="4" x="0.240594"  y="-0.240594"/>
+      <xacro:ball_caster_contact id="5" x="0.109092"  y="0.109092"/>
+      <xacro:ball_caster_contact id="6" x="-0.109092" y="0.109092"/>
+      <xacro:ball_caster_contact id="7" x="-0.109092" y="-0.109092"/>
+      <xacro:ball_caster_contact id="8" x="0.109092"  y="-0.109092"/>
+    </xacro:macro>
   <xacro:macro name="gimbalrotor_thrust_link" params="self rotor_direction">
     ## link

Commit message: flight check

File: robots/gimbalrotor/urdf/beetle_hyper/gimbalrotor.urdf.xacro (robot description, xacro)
@@ -25,5 +25,5 @@
         <origin xyz="0.0257171 0.0007358  0.0813823" rpy="0 0 0"/>
         <!-- <mass value="2.8200834"/> -->
-	<mass value="2.0200834"/>
+	<mass value="3.0200834"/>
         <inertia
             ixx="0.0679394" iyy="0.1142367" izz="0.1213159"
@@ -83,8 +83,8 @@
     </xacro:macro>
     ## dummy rotor arms
-    <xacro:dummy_rotor_arm id = "${child1}" x = "-0.12041" y="-0.12041" z = "0.0555" yaw = "${-pi*3/4.0}"/>
+    <xacro:dummy_rotor_arm id = "${child1}" x = "0.12041" y="0.12041" z = "0.0555" yaw = "${pi/4.0}"/>
     <xacro:dummy_rotor_arm id = "${child2}" x = "-0.12129" y="0.12150" z = "0.0555" yaw = "${pi*3.0/4.0}"/>
-    <xacro:dummy_rotor_arm id = "${child3}" x = "0.12129" y="-0.12150" z = "0.0555" yaw = "${-pi/4.0}"/>
-    <xacro:dummy_rotor_arm id = "${child4}" x = "0.12129" y="0.12150" z = "0.0555" yaw = "${pi/4.0}"/>
+    <xacro:dummy_rotor_arm id = "${child3}" x = "-0.12129" y="-0.12150" z = "0.0555" yaw = "${pi*5.0/4.0}"/>
+    <xacro:dummy_rotor_arm id = "${child4}" x = "0.12129" y="-0.12150" z = "0.0555" yaw = "${-pi/4.0}"/>
     ## dummy link for the contact point coordinate
       <link name="contact_point">
@@ -112,5 +112,5 @@
       <inertial>
         <origin xyz="0.0223521 0.0 0.00776312" rpy="0 0 0"/>
-p        <mass value="0.15944"/>
+        <mass value="0.15944"/>
         <inertia
             ixx="0.00007458" iyy="0.00007325" izz="0.00007756"
